Commit message: 完成仿真

File: src/sim_dog/edu_description/urdf/edu.urdf (robot description, URDF)
Before this commit: robot edu_urdf, 17 links, 16 joints
Links:
- added link laser, mass 0.125547937345628; visual mesh filename=package://edu_description/meshes/laser.STL
- link FL_ABAD_LINK: geometry collision box size=0.1 0.07 0.07; visual mesh filename=package://edu_description/meshes/FL_ABAD_LINK.STL
- link FL_FOOT_LINK: geometry collision sphere radius=0.02; visual mesh filename=package://edu_description/meshes/FL_FOOT_LINK.STL
- link FL_HIP_LINK: geometry collision box size=0.08392 0.17199 0.25400; visual mesh filename=package://edu_description/meshes/FL_HIP_LINK.STL
- link FL_KNEE_LINK: geometry collision box size=0.03481 0.02000 0.11477; visual mesh filename=package://edu_description/meshes/FL_KNEE_LINK.STL
- link FR_ABAD_LINK: geometry visual mesh filename=package://edu_description/meshes/FR_ABAD_LINK.STL
- link FR_FOOT_LINK: geometry collision sphere radius=0.02; visual mesh filename=package://edu_description/meshes/FR_FOOT_LINK.STL
- link FR_HIP_LINK: geometry visual mesh filename=package://edu_description/meshes/FR_HIP_LINK.STL
- link FR_KNEE_LINK: geometry visual mesh filename=package://edu_description/meshes/FR_KNEE_LINK.STL
- link RL_ABAD_LINK: geometry visual mesh filename=package://edu_description/meshes/RL_ABAD_LINK.STL
- link RL_FOOT_LINK: geometry collision sphere radius=0.02; visual mesh filename=package://edu_description/meshes/RL_FOOT_LINK.STL
- link RL_HIP_LINK: geometry visual mesh filename=package://edu_description/meshes/RL_HIP_LINK.STL
- link RL_KNEE_LINK: geometry visual mesh filename=package://edu_description/meshes/RL_KNEE_LINK.STL
- link RR_ABAD_LINK: geometry visual mesh filename=package://edu_description/meshes/RR_ABAD_LINK.STL
- link RR_FOOT_LINK: geometry collision sphere radius=0.02; visual mesh filename=package://edu_description/meshes/RR_FOOT_LINK.STL
- link RR_HIP_LINK: geometry visual mesh filename=package://edu_description/meshes/RR_HIP_LINK.STL
- link RR_KNEE_LINK: geometry visual mesh filename=package://edu_description/meshes/RR_KNEE_LINK.STL
- link base_link: geometry collision box size=0.4 0.1 0.05; visual mesh filename=package://edu_description/meshes/BASE_LINK.STL
Joints:
- added joint laser_joint: type fixed, parent base_link, child laser, origin xyz=0.21 0 0.1 rpy=0 0.2618 0, axis 0 0 0
- joint FL_ABAD_JOINT: limit lower=-0.4887 upper=0.4887 effort=0 velocity=0 -> lower=-0.4887 upper=0.4887 effort=48.0 velocity=28.0
- joint FL_HIP_JOINT: limit lower=-1.1519 upper=2.967 effort=0 velocity=0 -> lower=-1.1519 upper=2.967 effort=48.0 velocity=28.0
- joint FL_KNEE_JOINT: limit lower=-2.723 upper=-0.602 effort=0 velocity=0 -> lower=-2.723 upper=-0.602 effort=48.0 velocity=28.0
- joint FR_ABAD_JOINT: limit lower=-0.4887 upper=0.4887 effort=0 velocity=0 -> lower=-0.4887 upper=0.4887 effort=48.0 velocity=28.0
- joint FR_HIP_JOINT: limit lower=-1.1519 upper=2.967 effort=0 velocity=0 -> lower=-1.1519 upper=2.967 effort=48.0 velocity=28.0
- joint FR_KNEE_JOINT: limit lower=-2.723 upper=-0.602 effort=0 velocity=0 -> lower=-2.723 upper=-0.602 effort=48.0 velocity=28.0
- joint RL_ABAD_JOINT: limit lower=-0.4887 upper=0.4887 effort=0 velocity=0 -> lower=-0.4887 upper=0.4887 effort=48.0 velocity=28.0
- joint RL_HIP_JOINT: limit lower=-1.1519 upper=2.967 effort=0 velocity=0 -> lower=-1.1519 upper=2.967 effort=48.0 velocity=28.0
- joint RL_KNEE_JOINT: limit lower=-2.723 upper=-0.602 effort=0 velocity=0 -> lower=-2.723 upper=-0.602 effort=48.0 velocity=28.0
- joint RR_ABAD_JOINT: limit lower=-0.4887 upper=0.4887 effort=0 velocity=0 -> lower=-0.4887 upper=0.4887 effort=48.0 velocity=28.0
- joint RR_HIP_JOINT: limit lower=-1.1519 upper=2.967 effort=0 velocity=0 -> lower=-1.1519 upper=2.967 effort=48.0 velocity=28.0
- joint RR_KNEE_JOINT: limit lower=-2.723 upper=-0.602 effort=0 velocity=0 -> lower=-2.723 upper=-0.602 effort=48.0 velocity=28.0

Commit message: 新增深度相机

File: src/sim_dog/edu_description/urdf/edu.urdf (robot description, URDF)
Before this commit: robot edu_urdf, 18 links, 17 joints
Links:
- added link front_camera
Joints:
- added joint front_camera_joint: type fixed, parent base_link, child front_camera, origin xyz=0.26470 0 0.02038 rpy=0 0 0
